Commit message: panda description package update for gazebo simulation

File: src/panda_description/urdf/panda_arm.xacro (robot description, xacro)
@@ -3,5 +3,5 @@
   <xacro:macro name="panda_arm" params="arm_id:='panda' description_pkg:='panda_description' connected_to:='' xyz:='0 0 0' rpy:='0 0 0'">
     <xacro:unless value="${not connected_to}">
-      <joint name="${arm_id}_joint_${connected_to}" type="fixed">
+      <joint name="virtual_joint" type="fixed">
         <parent link="${connected_to}"/>
         <child link="${arm_id}_link0"/>

File: src/panda_description/urdf/panda_arm_hand.urdf.xacro (robot description, xacro)
@@ -6,5 +6,8 @@
   <xacro:include filename="$(find panda_description)/urdf/panda.gazebo.xacro"/>
   <xacro:panda_arm />
+  <xacro:panda_gazebo arm_id="panda"/>
+  <xacro:panda_arm xyz="0 0 0" rpy="0 0 0" connected_to="world"/>
   <xacro:hand ns="panda" rpy="0 0 ${-pi/4}" connected_to="panda_link8"/>
+  <link name="world" />
   <xacro:panda_gazebo robot_name="$(arg robot_name)" />
 </robot>
